File: pcb/TurboMaster-clean_noart.brd (EAGLE design)
At the start: 148 x 121.9 mm, 40 parts, among them IC1 74HCT244N, IC10 74HCT32N, IC11 74HCT244N, IC16 62256, IC17 62256, IC18 27C256, IC19 65C02, IC2 74HCT244N, IC3 74HCT374N, IC4 74HCT374N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

Commit message: Schematic signal naming updates
Connections:
- net !EN_$0001 renamed !EN_0001
- net !RAM1_CE renamed !CE_RAM1
- net !RAM1_WE renamed !WE_RAM1
- net !RAM2_CE renamed !CE_RAM2
- net !RAM2_WE renamed !WE_RAM2
- net !ROM_OE renamed !OE_ROM
- net !WRITE_$DXXX renamed !WR_DXXX
- net CLK_WRITE_$0000 renamed CLK_WR_0000
- net CLK_WRITE_$0001 renamed CLK_WR_0001
- net ROM_A13 renamed A13_ROM
- net ROM_A14 renamed A14_ROM
- net SEL_ROM renamed ROM_SEL
Changed lines of the file:
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@@
 <contactref element="IC14" pad="19"/>
 </signal>
-<signal name="ROM_A13">
+<signal name="A13_ROM">
 <wire x1="136.525" y1="-71.12" x2="134.62" y2="-73.025" width="0.254" layer="1"/>
 <wire x1="134.62" y1="-73.025" x2="106.68" y2="-73.025" width="0.254" layer="1"/>
@@
 <contactref element="IC18" pad="26"/>
 </signal>
-<signal name="ROM_A14">
+<signal name="A14_ROM">
 <wire x1="139.065" y1="-71.12" x2="135.89" y2="-74.295" width="0.254" layer="1"/>
 <wire x1="135.89" y1="-74.295" x2="107.95" y2="-74.295" width="0.254" layer="1"/>
@@
 <contactref element="IC15" pad="13"/>
 </signal>
-<signal name="!RAM1_CE">
+<signal name="!CE_RAM1">
 <wire x1="126.365" y1="-30.48" x2="126.365" y2="-22.86" width="0.254" layer="16"/>
 <wire x1="86.995" y1="-85.09" x2="88.9" y2="-86.995" width="0.254" layer="16"/>
@@
 <contactref element="IC10" pad="6"/>
 </signal>
-<signal name="!RAM1_WE">
+<signal name="!WE_RAM1">
 <wire x1="139.065" y1="-30.48" x2="139.065" y2="-24.13" width="0.254" layer="16"/>
 <wire x1="139.065" y1="-24.13" x2="140.335" y2="-22.86" width="0.254" layer="16"/>
@@
 <contactref element="IC12" pad="11"/>
 </signal>
-<signal name="!RAM2_WE">
+<signal name="!WE_RAM2">
 <wire x1="139.065" y1="-50.8" x2="139.065" y2="-46.99" width="0.254" layer="16"/>
 <wire x1="139.065" y1="-46.99" x2="143.51" y2="-42.545" width="0.254" layer="16"/>
@@
 <contactref element="IC17" pad="27"/>
 </signal>
-<signal name="!RAM2_CE">
+<signal name="!CE_RAM2">
 <wire x1="66.675" y1="1.27" x2="74.295" y2="1.27" width="0.254" layer="16"/>
 <wire x1="74.295" y1="1.27" x2="76.835" y2="3.81" width="0.254" layer="16"/>
@@
 <contactref element="IC15" pad="5"/>
 </signal>
-<signal name="!WRITE_$DXXX">
+<signal name="!WR_DXXX">
 <wire x1="66.675" y1="-6.35" x2="74.295" y2="-6.35" width="0.254" layer="16"/>
 <wire x1="103.505" y1="7.62" x2="102.235" y2="6.35" width="0.254" layer="16"/>
@@
 <contactref element="IC12" pad="1"/>
 </signal>
-<signal name="!EN_$0001">
+<signal name="!EN_0001">
 <wire x1="81.915" y1="-85.09" x2="81.915" y2="-83.185" width="0.254" layer="1"/>
 <wire x1="81.915" y1="-83.185" x2="81.28" y2="-82.55" width="0.254" layer="1"/>
@@
 <contactref element="IC12" pad="15"/>
 </signal>
-<signal name="CLK_WRITE_$0000">
+<signal name="CLK_WR_0000">
 <wire x1="79.375" y1="-85.09" x2="79.375" y2="-86.995" width="0.254" layer="1"/>
 <wire x1="79.375" y1="-86.995" x2="81.915" y2="-89.535" width="0.254" layer="1"/>
@@
 <contactref element="IC13" pad="12"/>
 </signal>
-<signal name="CLK_WRITE_$0001">
+<signal name="CLK_WR_0001">
 <wire x1="84.455" y1="-85.09" x2="84.455" y2="-87.63" width="0.254" layer="1"/>
 <wire x1="84.455" y1="-87.63" x2="85.725" y2="-88.9" width="0.254" layer="1"/>
@@
 <contactref element="IC12" pad="9"/>
 </signal>
-<signal name="SEL_ROM">
+<signal name="ROM_SEL">
 <contactref element="R6" pad="1"/>
 <wire x1="79.375" y1="-77.47" x2="76.835" y2="-74.93" width="0.254" layer="1"/>
@@
 <contactref element="IC15" pad="19"/>
 </signal>
-<signal name="!ROM_OE">
+<signal name="!OE_ROM">
 <wire x1="126.365" y1="-71.12" x2="126.365" y2="-69.85" width="0.254" layer="1"/>
 <wire x1="126.365" y1="-69.85" x2="128.905" y2="-67.31" width="0.254" layer="1"/>

Commit message: Working U1 and U4 JED files
Parts:
- renumbered IC12 to U4, IC13 to U1
Changed lines of the file:
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@@
 <element name="IC10" library="74xx-us-jlb" package="DIL14-RP" value="74HCT32N" x="94.615" y="11.43" rot="R270"/>
 <element name="IC19" library="commodore" package="DIL40-ROUNDPAD" value="65C02" x="95.885" y="-44.45" rot="R90"/>
-<element name="IC12" library="pal" package="DIL20-RP" value="" x="62.865" y="-7.62" rot="R270"/>
-<element name="IC13" library="pal" package="DIL20-RP" value="" x="88.265" y="-81.28" rot="R180"/>
+<element name="U4" library="pal" package="DIL20-RP" value="" x="62.865" y="-7.62" rot="R270"/>
+<element name="U1" library="pal" package="DIL20-RP" value="" x="88.265" y="-81.28" rot="R180"/>
 <element name="IC14" library="pal" package="DIL20-RP" value="" x="69.215" y="-60.96" rot="R180"/>
 <element name="IC15" library="pal" package="DIL20-RP" value="" x="107.315" y="11.43" rot="R270"/>
@@
 <contactref element="IC19" pad="1"/>
 <contactref element="IC19" pad="21"/>
-<contactref element="IC12" pad="10"/>
-<contactref element="IC13" pad="10"/>
+<contactref element="U4" pad="10"/>
+<contactref element="U1" pad="10"/>
 <contactref element="IC14" pad="10"/>
 <contactref element="IC15" pad="10"/>
@@
 <contactref element="IC10" pad="14"/>
 <contactref element="IC19" pad="8"/>
-<contactref element="IC12" pad="20"/>
-<contactref element="IC13" pad="20"/>
+<contactref element="U4" pad="20"/>
+<contactref element="U1" pad="20"/>
 <contactref element="IC14" pad="20"/>
 <contactref element="IC14" pad="4"/>
@@
 <wire x1="78.105" y1="-67.945" x2="78.105" y2="-64.77" width="0.254" layer="1"/>
 <contactref element="IC19" pad="2"/>
-<contactref element="IC13" pad="17"/>
+<contactref element="U1" pad="17"/>
 <contactref element="IC14" pad="19"/>
 </signal>
@@
 <wire x1="106.045" y1="-81.28" x2="106.045" y2="-73.66" width="0.254" layer="1"/>
 <wire x1="106.045" y1="-73.66" x2="106.68" y2="-73.025" width="0.254" layer="1"/>
-<contactref element="IC13" pad="18"/>
+<contactref element="U1" pad="18"/>
 <contactref element="IC18" pad="26"/>
 </signal>
@@
 <wire x1="107.95" y1="-74.295" x2="107.315" y2="-74.93" width="0.254" layer="1"/>
 <wire x1="107.315" y1="-74.93" x2="107.315" y2="-83.185" width="0.254" layer="1"/>
-<contactref element="IC13" pad="19"/>
+<contactref element="U1" pad="19"/>
 <contactref element="IC18" pad="27"/>
 </signal>
@@
 <contactref element="IC9" pad="13"/>
 <contactref element="IC19" pad="40"/>
-<contactref element="IC13" pad="4"/>
+<contactref element="U1" pad="4"/>
 <contactref element="X1" pad="C"/>
 <wire x1="2.8702" y1="21.59" x2="29.5275" y2="21.59" width="0.254" layer="16"/>
@@
 <wire x1="88.265" y1="-63.5" x2="93.345" y2="-68.58" width="0.254" layer="1"/>
 <contactref element="IC19" pad="38"/>
-<contactref element="IC13" pad="16"/>
+<contactref element="U1" pad="16"/>
 </signal>
 <signal name="PHI0">
@@
 <wire x1="72.39" y1="1.905" x2="73.025" y2="2.54" width="0.254" layer="1"/>
 <contactref element="IC19" pad="37"/>
-<contactref element="IC12" pad="2"/>
-<contactref element="IC13" pad="3"/>
+<contactref element="U4" pad="2"/>
+<contactref element="U1" pad="3"/>
 <contactref element="IC15" pad="13"/>
 </signal>
@@
 <via x="140.335" y="-48.26" extent="1-16" drill="0.3048"/>
 <contactref element="IC10" pad="9"/>
-<contactref element="IC13" pad="15"/>
+<contactref element="U1" pad="15"/>
 <contactref element="IC16" pad="22"/>
 </signal>
@@
 <contactref element="IC10" pad="13"/>
 <contactref element="IC19" pad="34"/>
-<contactref element="IC12" pad="11"/>
+<contactref element="U4" pad="11"/>
 </signal>
 <signal name="!WE_RAM2">
@@
 <via x="139.065" y="-40.64" extent="1-16" drill="0.3048"/>
 <contactref element="IC10" pad="12"/>
-<contactref element="IC12" pad="19"/>
+<contactref element="U4" pad="19"/>
 <contactref element="IC17" pad="22"/>
 </signal>
@@
 <wire x1="95.885" y1="-3.81" x2="95.885" y2="-4.445" width="0.254" layer="16"/>
 <wire x1="95.885" y1="-4.445" x2="97.79" y2="-6.35" width="0.254" layer="16"/>
-<contactref element="IC12" pad="16"/>
+<contactref element="U4" pad="16"/>
 <contactref element="IC15" pad="7"/>
 </signal>
@@
 <via x="107.95" y="10.795" extent="1-16" drill="0.3048"/>
 <contactref element="IC8" pad="6"/>
-<contactref element="IC12" pad="1"/>
+<contactref element="U4" pad="1"/>
 </signal>
 <signal name="!EN_0001">
@@
 <via x="146.685" y="-83.82" extent="1-16" drill="0.3048"/>
 <contactref element="IC8" pad="1"/>
-<contactref element="IC13" pad="13"/>
+<contactref element="U1" pad="13"/>
 </signal>
 <signal name="!=00000000000000XX">
@@
 <wire x1="128.905" y1="-91.44" x2="128.905" y2="-83.82" width="0.254" layer="16"/>
 <contactref element="IC7" pad="19"/>
-<contactref element="IC13" pad="11"/>
+<contactref element="U1" pad="11"/>
 </signal>
 <signal name="!=000000XXXXXXXXXX">
@@
 <wire x1="143.51" y1="-76.2" x2="145.0975" y2="-74.6125" width="0.254" layer="16"/>
 <contactref element="IC7" pad="1"/>
-<contactref element="IC12" pad="15"/>
+<contactref element="U4" pad="15"/>
 </signal>
 <signal name="CLK_WR_0000">
@@
 <via x="145.415" y="-81.28" extent="1-16" drill="0.3048"/>
 <contactref element="IC9" pad="11"/>
-<contactref element="IC13" pad="12"/>
+<contactref element="U1" pad="12"/>
 </signal>
 <signal name="CLK_WR_0001">
@@
 <via x="142.875" y="-81.28" extent="1-16" drill="0.3048"/>
 <contactref element="IC8" pad="11"/>
-<contactref element="IC13" pad="14"/>
+<contactref element="U1" pad="14"/>
 </signal>
 <signal name="!FLAG_CHAREN">
@@
 <via x="108.585" y="-1.27" extent="1-16" drill="0.3048"/>
 <contactref element="IC8" pad="9"/>
-<contactref element="IC12" pad="18"/>
+<contactref element="U4" pad="18"/>
 </signal>
 <signal name="!FLAG_LORAM">
@@
 <via x="131.445" y="22.225" extent="1-16" drill="0.3048"/>
 <contactref element="IC8" pad="5"/>
-<contactref element="IC12" pad="9"/>
+<contactref element="U4" pad="9"/>
 </signal>
 <signal name="ROM_SEL">
@@
 <wire x1="67.945" y1="-72.39" x2="70.485" y2="-74.93" width="0.254" layer="1"/>
 <wire x1="70.485" y1="-74.93" x2="76.835" y2="-74.93" width="0.254" layer="1"/>
-<contactref element="IC13" pad="9"/>
+<contactref element="U1" pad="9"/>
 <contactref element="S1" pad="9"/>
 </signal>
@@
 <wire x1="78.105" y1="19.685" x2="78.74" y2="19.05" width="0.254" layer="1"/>
 <contactref element="IC11" pad="1"/>
-<contactref element="IC13" pad="8"/>
+<contactref element="U1" pad="8"/>
 <contactref element="S1" pad="8"/>
 </signal>
@@
 <via x="142.875" y="-3.81" extent="1-16" drill="0.3048"/>
 <wire x1="142.875" y1="-3.81" x2="144.145" y2="-3.81" width="0.254" layer="16"/>
-<contactref element="IC12" pad="14"/>
+<contactref element="U4" pad="14"/>
 <contactref element="IC18" pad="22"/>
 </signal>
@@
 <contactref element="IC4" pad="8"/>
 <contactref element="IC19" pad="9"/>
-<contactref element="IC13" pad="2"/>
+<contactref element="U1" pad="2"/>
 <contactref element="IC18" pad="10"/>
 <contactref element="IC16" pad="10"/>
@@
 <contactref element="IC4" pad="13"/>
 <contactref element="IC19" pad="10"/>
-<contactref element="IC13" pad="1"/>
+<contactref element="U1" pad="1"/>
 <contactref element="IC18" pad="9"/>
 <contactref element="IC16" pad="9"/>
@@
 <contactref element="IC3" pad="14"/>
 <contactref element="IC19" pad="19"/>
-<contactref element="IC12" pad="8"/>
+<contactref element="U4" pad="8"/>
 <contactref element="IC18" pad="21"/>
 <contactref element="IC16" pad="21"/>
@@
 <contactref element="IC3" pad="7"/>
 <contactref element="IC19" pad="20"/>
-<contactref element="IC12" pad="7"/>
+<contactref element="U4" pad="7"/>
 <contactref element="IC18" pad="23"/>
 <contactref element="IC16" pad="23"/>
@@
 <contactref element="IC3" pad="4"/>
 <contactref element="IC19" pad="22"/>
-<contactref element="IC12" pad="6"/>
+<contactref element="U4" pad="6"/>
 <contactref element="IC18" pad="2"/>
 <contactref element="IC16" pad="2"/>
@@
 <contactref element="IC3" pad="17"/>
 <contactref element="IC19" pad="23"/>
-<contactref element="IC12" pad="5"/>
-<contactref element="IC13" pad="7"/>
+<contactref element="U4" pad="5"/>
+<contactref element="U1" pad="7"/>
 <contactref element="IC16" pad="26"/>
 <contactref element="IC17" pad="26"/>
@@
 <contactref element="IC3" pad="18"/>
 <contactref element="IC19" pad="24"/>
-<contactref element="IC12" pad="4"/>
-<contactref element="IC13" pad="6"/>
+<contactref element="U4" pad="4"/>
+<contactref element="U1" pad="6"/>
 <contactref element="IC16" pad="1"/>
 <contactref element="IC17" pad="1"/>
@@
 <contactref element="IC3" pad="3"/>
 <contactref element="IC19" pad="25"/>
-<contactref element="IC12" pad="3"/>
-<contactref element="IC13" pad="5"/>
+<contactref element="U4" pad="3"/>
+<contactref element="U1" pad="5"/>
 </signal>
 <signal name="D0">
@@
 <wire x1="75.565" y1="-2.54" x2="74.295" y2="-3.81" width="0.254" layer="1"/>
 <via x="74.295" y="-3.81" extent="1-16" drill="0.3048"/>
-<contactref element="IC12" pad="17"/>
+<contactref element="U4" pad="17"/>
 <contactref element="IC15" pad="4"/>
 </signal>
