File: pcb/TurboMaster-clean_noart.sch (EAGLE design)
At the start: 40 parts, among them IC1 74HCT244N, IC10 74HCT32N, IC11 74HCT244N, IC16 62256, IC17 62256, IC18 27C256, IC19 65C02, IC2 74HCT244N, IC3 74HCT374N, IC4 74HCT374N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

Commit message: Schematic signal naming updates
Connections:
- net !EN_$0001 renamed !EN_0001
- net !RAM1_CE renamed !CE_RAM1
- net !RAM1_WE renamed !WE_RAM1
- net !RAM2_CE renamed !CE_RAM2
- net !RAM2_WE renamed !WE_RAM2
- net !ROM_OE renamed !OE_ROM
- net !WRITE_$DXXX renamed !WR_DXXX
- net CLK_WRITE_$0000 renamed CLK_WR_0000
- net CLK_WRITE_$0001 renamed CLK_WR_0001
- net ROM_A13 renamed A13_ROM
- net ROM_A14 renamed A14_ROM
- net SEL_ROM renamed ROM_SEL
Other:
- note added: "U1: CLK_WR_0 = A0 + A1 + nEQ000X + nRESET' + PHI0' ; nEN_0001 = nEQ000X + nRESET' + PHI0' ; CLK_WR_1 = A0' + A1 + nEQ000X + nRESET' + PHI0' ; nCE_ROM1 = A15 + PHI0' ; nSO = 1; nRDY = nDISABLE' ; A13_ROM = A14 ROM_SEL' + A14 A13' ; A14_ROM = A14 A13 ;"
- note added: "U4 (optimized): O2 = PHI0' + A15' + R/W' + /HIRAM' A13 + A14' A13' + A13' A12' + /HIRAM' /LORAM' + A14' /LORAM' + A13' /CHAREN; O3 = not(!A15 & !A14 & !A13 & !A12 & !A11 & !A10 & !R/W); O4 = not(!R/W & PHI0 & !(A15 & A14 & !A13 & A12)) O5 = not(_HIRAM | _LORAM) & A15 & A14 & !A13 & A12 & _CHAREN); O7 = not(PHI0 & A15 & (!/HIRAM | !A14 | !A13 | !R/W) & (!/HIRAM | !A14 | !A12 | !R/W) & (!/HIRAM | !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"
- note added: "U4: O0 = 1; O1 = 1; O2 = PHI0' + A15' + R/W' + /HIRAM' A13 + A14' A13' + A13' A12' + /HIRAM' /LORAM' + A14' /LORAM' + A13' /CHAREN; O3 = A15 + A14 + A13 + A12 + A11 + A10 + R/W ; O4 = PHI0' + R/W + A15 A14 A13' A12 /CHAREN' + /HIRAM' A15 A14 A13' A12 /LORAM' ; O5 = PHI0' + A15' + A14' + A13 + A12' + /CHAREN' + /HIRAM' /LORAM' ; O7 = PHI0' + A15' + /HIRAM A14 A13 R/W + /HIRAM A14 A12 R/W + /HIRAM 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"
- note removed: "IC12 (optimized): O2 = PHI0' + A15' + R/W' + /HIRAM' A13 + A14' A13' + A13' A12' + /HIRAM' /LORAM' + A14' /LORAM' + A13' /CHAREN; O3 = not(!A15 & !A14 & !A13 & !A12 & !A11 & !A10 & !R/W); O4 = not(!R/W & PHI0 & !(A15 & A14 & !A13 & A12)) O5 = not(_HIRAM | _LORAM) & A15 & A14 & !A13 & A12 & _CHAREN); O7 = not(PHI0 & A15 & (!/HIRAM | !A14 | !A13 | !R/W) & (!/HIRAM | !A14 | !A12 | !R/W) & (!/HIRAM |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"
- note removed: "IC12: O0 = 1; O1 = 1; O2 = PHI0' + A15' + R/W' + /HIRAM' A13 + A14' A13' + A13' A12' + /HIRAM' /LORAM' + A14' /LORAM' + A13' /CHAREN; O3 = A15 + A14 + A13 + A12 + A11 + A10 + R/W ; O4 = PHI0' + R/W + A15 A14 A13' A12 /CHAREN' + /HIRAM' A15 A14 A13' A12 /LORAM' ; O5 = PHI0' + A15' + A14' + A13 + A12' + /CHAREN' + /HIRAM' /LORAM' ; O7 = PHI0' + A15' + /HIRAM A14 A13 R/W + /HIRAM A14 A12 R/W + /HIRA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"
- note removed: "IC13: O0 = A1 + A0 + PHI0' + /RESET' + /eq000X; O1 = PHI0' + /RESET' + /eq000X; O2 = A1 + A0' + PHI0' + /RESET' + /eq000X; O3 = PHI0' + A15 ; O4 = 1; O5 = DISABLE' ; O6 = A14 A13' + A14 SEL_ROM' ; O7 = A14 A13 ;"

Commit message: Working U1 and U4 JED files
Parts:
- renumbered IC12 to U4, IC13 to U1
Changed lines of the file:
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@@
 <part name="IC10" library="74xx-us-jlb" deviceset="74*32" device="N" technology="HCT"/>
 <part name="IC19" library="commodore" deviceset="65*02" device="-RP" technology="C" value="65C02"/>
-<part name="IC12" library="pal" deviceset="16L8" device="-RP"/>
-<part name="IC13" library="pal" deviceset="16L8" device="-RP"/>
+<part name="U4" library="pal" deviceset="16L8" device="-RP"/>
+<part name="U1" library="pal" deviceset="16L8" device="-RP"/>
 <part name="IC14" library="pal" deviceset="16R4" device="-RP"/>
 <part name="IC15" library="pal" deviceset="16R6" device="-RP"/>
@@
 <instance part="IC10" gate="D" x="134.62" y="203.2"/>
 <instance part="IC19" gate="A" x="233.68" y="368.3"/>
-<instance part="IC12" gate="G$1" x="134.62" y="177.8"/>
-<instance part="IC13" gate="G$1" x="134.62" y="142.24"/>
+<instance part="U4" gate="G$1" x="134.62" y="177.8"/>
+<instance part="U1" gate="G$1" x="134.62" y="142.24"/>
 <instance part="IC14" gate="G$1" x="134.62" y="104.14"/>
 <instance part="IC15" gate="G$1" x="134.62" y="63.5"/>
@@
 <wire x1="147.32" y1="139.7" x2="162.56" y2="139.7" width="0.1524" layer="91"/>
 <label x="162.56" y="139.7" size="1.27" layer="95" xref="yes"/>
-<pinref part="IC13" gate="G$1" pin="O5"/>
+<pinref part="U1" gate="G$1" pin="O5"/>
 </segment>
 </net>
@@
 <wire x1="147.32" y1="137.16" x2="162.56" y2="137.16" width="0.1524" layer="91"/>
 <label x="162.56" y="137.16" size="1.27" layer="95" xref="yes"/>
-<pinref part="IC13" gate="G$1" pin="O6"/>
+<pinref part="U1" gate="G$1" pin="O6"/>
 </segment>
 </net>
@@
 <wire x1="147.32" y1="134.62" x2="162.56" y2="134.62" width="0.1524" layer="91"/>
 <label x="162.56" y="134.62" size="1.27" layer="95" xref="yes"/>
-<pinref part="IC13" gate="G$1" pin="O7"/>
+<pinref part="U1" gate="G$1" pin="O7"/>
 </segment>
 </net>
@@
 <wire x1="121.92" y1="144.78" x2="106.68" y2="144.78" width="0.1524" layer="91"/>
 <label x="106.68" y="144.78" size="1.27" layer="95" rot="R180" xref="yes"/>
-<pinref part="IC13" gate="G$1" pin="I3"/>
+<pinref part="U1" gate="G$1" pin="I3"/>
 </segment>
 </net>
@@
 <wire x1="147.32" y1="142.24" x2="162.56" y2="142.24" width="0.1524" layer="91"/>
 <label x="162.56" y="142.24" size="1.27" layer="95" xref="yes"/>
-<pinref part="IC13" gate="G$1" pin="O4"/>
+<pinref part="U1" gate="G$1" pin="O4"/>
 </segment>
 </net>
@@
 <wire x1="121.92" y1="147.32" x2="106.68" y2="147.32" width="0.1524" layer="91"/>
 <label x="106.68" y="147.32" size="1.27" layer="95" rot="R180" xref="yes"/>
-<pinref part="IC13" gate="G$1" pin="I2"/>
+<pinref part="U1" gate="G$1" pin="I2"/>
 </segment>
 <segment>
@@
 <wire x1="121.92" y1="185.42" x2="106.68" y2="185.42" width="0.1524" layer="91"/>
 <label x="106.68" y="185.42" size="1.27" layer="95" rot="MR0" xref="yes"/>
-<pinref part="IC12" gate="G$1" pin="I1"/>
+<pinref part="U4" gate="G$1" pin="I1"/>
 </segment>
 </net>
@@
 <wire x1="147.32" y1="144.78" x2="162.56" y2="144.78" width="0.1524" layer="91"/>
 <label x="162.56" y="144.78" size="1.27" layer="95" xref="yes"/>
-<pinref part="IC13" gate="G$1" pin="O3"/>
+<pinref part="U1" gate="G$1" pin="O3"/>
 </segment>
 <segment>
@@
 <wire x1="121.92" y1="165.1" x2="111.76" y2="165.1" width="0.1524" layer="91"/>
 <label x="106.68" y="162.56" size="1.27" layer="95" rot="MR0" xref="yes"/>
-<pinref part="IC12" gate="G$1" pin="I9"/>
+<pinref part="U4" gate="G$1" pin="I9"/>
 </segment>
 </net>
@@
 <wire x1="147.32" y1="170.18" x2="162.56" y2="170.18" width="0.1524" layer="91"/>
 <label x="162.56" y="170.18" size="1.27" layer="95" xref="yes"/>
-<pinref part="IC12" gate="G$1" pin="O7"/>
+<pinref part="U4" gate="G$1" pin="O7"/>
 </segment>
 <segment>
@@
 <wire x1="147.32" y1="177.8" x2="162.56" y2="177.8" width="0.1524" layer="91"/>
 <label x="162.56" y="177.8" size="1.27" layer="95" xref="yes"/>
-<pinref part="IC12" gate="G$1" pin="O4"/>
+<pinref part="U4" gate="G$1" pin="O4"/>
 </segment>
 <segment>
@@
 <wire x1="121.92" y1="187.96" x2="106.68" y2="187.96" width="0.1524" layer="91"/>
 <label x="106.68" y="187.96" size="1.27" layer="95" rot="MR0" xref="yes"/>
-<pinref part="IC12" gate="G$1" pin="I0"/>
+<pinref part="U4" gate="G$1" pin="I0"/>
 </segment>
 </net>
@@
 <wire x1="147.32" y1="149.86" x2="162.56" y2="149.86" width="0.1524" layer="91"/>
 <label x="162.56" y="149.86" size="1.27" layer="95" xref="yes"/>
-<pinref part="IC13" gate="G$1" pin="O1"/>
+<pinref part="U1" gate="G$1" pin="O1"/>
 </segment>
 </net>
@@
 <wire x1="114.3" y1="127" x2="106.68" y2="127" width="0.1524" layer="91"/>
 <label x="106.68" y="127" size="1.27" layer="95" rot="R180" xref="yes"/>
-<pinref part="IC13" gate="G$1" pin="I9"/>
+<pinref part="U1" gate="G$1" pin="I9"/>
 </segment>
 </net>
@@
 <wire x1="147.32" y1="180.34" x2="162.56" y2="180.34" width="0.1524" layer="91"/>
 <label x="162.56" y="180.34" size="1.27" layer="95" xref="yes"/>
-<pinref part="IC12" gate="G$1" pin="O3"/>
+<pinref part="U4" gate="G$1" pin="O3"/>
 </segment>
 </net>
@@
 <wire x1="147.32" y1="152.4" x2="162.56" y2="152.4" width="0.1524" layer="91"/>
 <label x="162.56" y="152.4" size="1.27" layer="95" xref="yes"/>
-<pinref part="IC13" gate="G$1" pin="O0"/>
+<pinref part="U1" gate="G$1" pin="O0"/>
 </segment>
 <segment>
@@
 <wire x1="147.32" y1="147.32" x2="162.56" y2="147.32" width="0.1524" layer="91"/>
 <label x="162.56" y="147.32" size="1.27" layer="95" xref="yes"/>
-<pinref part="IC13" gate="G$1" pin="O2"/>
+<pinref part="U1" gate="G$1" pin="O2"/>
 </segment>
 </net>
@@
 <wire x1="147.32" y1="172.72" x2="162.56" y2="172.72" width="0.1524" layer="91"/>
 <label x="162.56" y="172.72" size="1.27" layer="95" xref="yes"/>
-<pinref part="IC12" gate="G$1" pin="O6"/>
+<pinref part="U4" gate="G$1" pin="O6"/>
 </segment>
 </net>
@@
 <wire x1="121.92" y1="167.64" x2="109.22" y2="167.64" width="0.1524" layer="91"/>
 <label x="106.68" y="165.1" size="1.27" layer="95" rot="MR0" xref="yes"/>
-<pinref part="IC12" gate="G$1" pin="I8"/>
+<pinref part="U4" gate="G$1" pin="I8"/>
 </segment>
 </net>
@@
 <wire x1="111.76" y1="129.54" x2="106.68" y2="129.54" width="0.1524" layer="91"/>
 <label x="106.68" y="129.54" size="1.27" layer="95" rot="R180" xref="yes"/>
-<pinref part="IC13" gate="G$1" pin="I8"/>
+<pinref part="U1" gate="G$1" pin="I8"/>
 </segment>
 </net>
@@
 <wire x1="109.22" y1="132.08" x2="106.68" y2="132.08" width="0.1524" layer="91"/>
 <label x="106.68" y="132.08" size="1.27" layer="95" rot="R180" xref="yes"/>
-<pinref part="IC13" gate="G$1" pin="I7"/>
+<pinref part="U1" gate="G$1" pin="I7"/>
 </segment>
 <segment>
@@
 <wire x1="147.32" y1="182.88" x2="162.56" y2="182.88" width="0.1524" layer="91"/>
 <label x="162.56" y="182.88" size="1.27" layer="95" xref="yes"/>
-<pinref part="IC12" gate="G$1" pin="O2"/>
+<pinref part="U4" gate="G$1" pin="O2"/>
 </segment>
 <segment>
@@
 <wire x1="106.68" y1="152.4" x2="109.22" y2="149.86" width="0.1524" layer="91"/>
 <label x="109.22" y="149.86" size="1.778" layer="95"/>
-<pinref part="IC13" gate="G$1" pin="I1"/>
+<pinref part="U1" gate="G$1" pin="I1"/>
 </segment>
 <segment>
@@
 <wire x1="106.68" y1="154.94" x2="109.22" y2="152.4" width="0.1524" layer="91"/>
 <label x="109.22" y="152.4" size="1.778" layer="95"/>
-<pinref part="IC13" gate="G$1" pin="I0"/>
+<pinref part="U1" gate="G$1" pin="I0"/>
 </segment>
 <segment>
@@
 <wire x1="109.22" y1="170.18" x2="121.92" y2="170.18" width="0.1524" layer="91"/>
 <label x="109.22" y="170.18" size="1.778" layer="95"/>
-<pinref part="IC12" gate="G$1" pin="I7"/>
+<pinref part="U4" gate="G$1" pin="I7"/>
 </segment>
 <segment>
@@
 <wire x1="109.22" y1="172.72" x2="121.92" y2="172.72" width="0.1524" layer="91"/>
 <label x="109.22" y="172.72" size="1.778" layer="95"/>
-<pinref part="IC12" gate="G$1" pin="I6"/>
+<pinref part="U4" gate="G$1" pin="I6"/>
 </segment>
 <segment>
@@
 <wire x1="109.22" y1="175.26" x2="121.92" y2="175.26" width="0.1524" layer="91"/>
 <label x="109.22" y="175.26" size="1.778" layer="95"/>
-<pinref part="IC12" gate="G$1" pin="I5"/>
+<pinref part="U4" gate="G$1" pin="I5"/>
 </segment>
 <segment>
@@
 <wire x1="109.22" y1="177.8" x2="121.92" y2="177.8" width="0.1524" layer="91"/>
 <label x="109.22" y="177.8" size="1.778" layer="95"/>
-<pinref part="IC12" gate="G$1" pin="I4"/>
+<pinref part="U4" gate="G$1" pin="I4"/>
 </segment>
 <segment>
@@
 <wire x1="109.22" y1="137.16" x2="121.92" y2="137.16" width="0.1524" layer="91"/>
 <label x="109.22" y="137.16" size="1.778" layer="95"/>
-<pinref part="IC13" gate="G$1" pin="I6"/>
+<pinref part="U1" gate="G$1" pin="I6"/>
 </segment>
 <segment>
@@
 <wire x1="109.22" y1="180.34" x2="121.92" y2="180.34" width="0.1524" layer="91"/>
 <label x="109.22" y="180.34" size="1.778" layer="95"/>
-<pinref part="IC12" gate="G$1" pin="I3"/>
+<pinref part="U4" gate="G$1" pin="I3"/>
 </segment>
 <segment>
@@
 <wire x1="109.22" y1="139.7" x2="121.92" y2="139.7" width="0.1524" layer="91"/>
 <label x="109.22" y="139.7" size="1.778" layer="95"/>
-<pinref part="IC13" gate="G$1" pin="I5"/>
+<pinref part="U1" gate="G$1" pin="I5"/>
 </segment>
 <segment>
@@
 <wire x1="109.22" y1="182.88" x2="121.92" y2="182.88" width="0.1524" layer="91"/>
 <label x="109.22" y="182.88" size="1.778" layer="95"/>
-<pinref part="IC12" gate="G$1" pin="I2"/>
+<pinref part="U4" gate="G$1" pin="I2"/>
 </segment>
 <segment>
@@
 <wire x1="109.22" y1="142.24" x2="121.92" y2="142.24" width="0.1524" layer="91"/>
 <label x="109.22" y="142.24" size="1.778" layer="95"/>
-<pinref part="IC13" gate="G$1" pin="I4"/>
+<pinref part="U1" gate="G$1" pin="I4"/>
 </segment>
 <segment>
@@
 <wire x1="147.32" y1="175.26" x2="162.56" y2="175.26" width="0.1524" layer="91"/>
 <label x="162.56" y="175.26" size="1.27" layer="95" xref="yes"/>
-<pinref part="IC12" gate="G$1" pin="O5"/>
-</segment>
-<segment>
+<pinref part="U4" gate="G$1" pin="O5"/>
+</segment>
+<segment>
